File: CAN-SnifferPCB.kicad_pcb (KiCad board)
At the start: 2 copper layers, 70 x 50 mm, 29 parts, among them J1 CANConnIn, J2 CANConnOut, U1 Nucleo_L432KC, U2 ADM3055E, U3 CDSOT23-T24CAN

Commit message: Adds Terminating resistor label
Other:
- board text added: "Resistors"
- board text added: "Terminating"
